Commit message: chore: cambio a color gris a la mesa

File: src/npam_robot_description/urdf/npam_robot_macro.xacro (robot description, xacro)
@@ -22,4 +22,7 @@
         </geometry>
         <origin xyz="0 0 0" rpy="0 0 ${pi}"/>
+        <material name="GreyMetallic">
+          <color rgba="0.7 0.7 0.7 1.0"/>
+        </material>
       </visual>
       <collision>
