Commit message: FEAT: Funcionalidad basica de RViz

File: src/Universal_Robots_ROS2_Description/urdf/ur_macro.xacro (robot description, xacro)
@@ -417,4 +417,37 @@
       <origin xyz="0 0 0" rpy="${pi} 0 0"/>
     </joint>
+    <!-- |||||||||||||||||||||||||||||||||||||||||||||||||||||||||||||||||||||||||||||||||||||||||||||||||||||||||||||||||||||| -->
+    <link name="mesa">
+      <visual>
+        <origin xyz="0 0 0" rpy="0 0 ${pi}"/>
+        <geometry>
+          <mesh filename="file://$(find ur_description)/meshes/Escenas/estacion_sobredimensionada.stl" scale="0.001 0.001 0.001"/>
+        </geometry>
+        <material name="GreyMetallic">
+          <color rgba="0.7 0.7 0.7 1.0"/>
+        </material>
+      </visual>
+      <collision>
+        <origin xyz="0 0 0" rpy="0 0 ${pi}"/>
+        <geometry>
+          <mesh filename="file://$(find ur_description)/meshes/Escenas/estacion_sobredimensionada.stl" scale="0.001 0.001 0.001"/>
+        </geometry>
+      </collision>
+    <!-- |||||||||||||||||||||||||||||||||||||||||||||||||||||||||||||||||||||||||||||||||||||||||||||||||||||||||||||||||||||| -->
+    </link>
+        <joint name="plataforma" type="fixed">
+      <parent link="${tf_prefix}base_link" />
+      <child link="mesa" />
+      <origin xyz="0.76884 -0.27794 -0.16726" rpy="-0.0054 -0.0053 0.0116"/>
+      <axis xyz="0 0 1" />
+    </joint>
+    <!-- <joint name="cama_impresion" type="fixed">
+      <parent link="${tf_prefix}wrist_3_link" />
+      <child link="cama_impresion" />
+      <origin xyz="0 0 0.25" rpy="0 ${-pi/2} ${-pi/2-0.1}" />
+      <axis xyz="0 0 1" />
+    </joint>
+     -->
+    <!-- |||||||||||||||||||||||||||||||||||||||||||||||||||||||||||||||||||||||||||||||||||||||||||||||||||||||||||||||||||||| -->
     <!-- ROS-Industrial 'base' frame - base_link to UR 'Base' Coordinates transform -->
     <link name="${tf_prefix}base"/>

Commit message: FEAT: Test con barrera, punto A y B en Moveit planner, organizacion del paquete general

File: src/Universal_Robots_ROS2_Description/urdf/ur_macro.xacro (robot description, xacro)
@@ -83,5 +83,6 @@
     trajectory_port:=50003
     non_blocking_read:=true
-    keep_alive_count:=2"
+    keep_alive_count:=2
+    pruebas:=false"
     >
     <!-- Load configuration data from the provided .yaml files -->
@@ -434,7 +435,29 @@
         </geometry>
       </collision>
+    </link>
+    <link name="${tf_prefix}cama_impresion">
+      <visual>
+        <origin xyz="0 0 0" rpy="0 ${-pi/2} 0 "/>
+        <geometry>
+          <mesh filename="file://$(find ur_description)/meshes/Escenas/Camas/cama_impresion.stl" scale="0.001 0.001 0.001"/>
+        </geometry>
+        <material name="White">
+        <color rgba="1 1 1 1.0"/>
+      </material>
+      </visual>
+      <collision>
+        <origin xyz="0 0 0" rpy="0 ${-pi/2} 0"/>
+        <geometry>
+          <mesh filename="file://$(find ur_description)/meshes/Escenas/Camas/cama_impresion.stl" scale="0.001 0.001 0.001"/>
+        </geometry>
+      </collision>
+      <inertial>
+        <origin xyz="0 0 0" rpy="0 0 0"/>
+        <mass value="${wrist_3_mass}"/>
+        <inertia ixx="0.00079" ixy="0.0" ixz="0.0" iyy="0.00079" iyz="0.0" izz="0.00034"/>
+      </inertial>
+    </link>
     <!-- |||||||||||||||||||||||||||||||||||||||||||||||||||||||||||||||||||||||||||||||||||||||||||||||||||||||||||||||||||||| -->
-    </link>
-        <joint name="plataforma" type="fixed">
+    <joint name="plataforma" type="fixed">
       <parent link="${tf_prefix}base_link" />
       <child link="mesa" />
@@ -442,11 +465,4 @@
       <axis xyz="0 0 1" />
     </joint>
-    <!-- <joint name="cama_impresion" type="fixed">
-      <parent link="${tf_prefix}wrist_3_link" />
-      <child link="cama_impresion" />
-      <origin xyz="0 0 0.25" rpy="0 ${-pi/2} ${-pi/2-0.1}" />
-      <axis xyz="0 0 1" />
-    </joint>
-     -->
     <!-- |||||||||||||||||||||||||||||||||||||||||||||||||||||||||||||||||||||||||||||||||||||||||||||||||||||||||||||||||||||| -->
     <!-- ROS-Industrial 'base' frame - base_link to UR 'Base' Coordinates transform -->
@@ -477,4 +493,34 @@
       <child link="${tf_prefix}tool0"/>
     </joint>
+  <!-- |||||||||||||||||||||||||||||||||||||||||||||||||||||||||||||||||||||||||||||||||||||||||||||||||||||||||||||||||||||| -->
+    <joint name="${tf_prefix}ft_to_cama_impresion_joint" type="fixed">
+      <parent link="${tf_prefix}tool0" />
+      <child link="${tf_prefix}cama_impresion" />
+      <origin xyz="0 0 0.167" rpy="0 0 0" />
+      <axis xyz="0 0 1" />
+    </joint>
+  <!-- |||||||||||||||||||||||||||||||||||||||||||||||||||||||||||||||||||||||||||||||||||||||||||||||||||||||||||||||||||||| -->
+    <!-- <link name="barrier_link">
+      <visual>
+        <origin xyz="0 0 0" rpy="0 0 0"/>
+        <geometry>
+          <box size="3 0.005 0.5" />
+        </geometry>
+        <material name="BarrierColor">
+          <color rgba="1.0 1.0 0.0 1.0"/>
+        </material>
+      </visual>
+      <collision>
+        <origin xyz="0 0 0" rpy="0 0 0"/>
+        <geometry>
+          <box size="3 0.005 0.5" />
+        </geometry>
+      </collision>
+    </link>
+    <joint name="barrier_joint" type="fixed">
+      <parent link="${tf_prefix}base_link"/>
+      <child link="barrier_link"/>
+      <origin xyz="0 -1.15 0.5" rpy="0 0 0"/>
+    </joint> -->
   </xacro:macro>
 </robot>

File: src/Universal_Robots_ROS2_Driver/ur_moveit_config/srdf/ur_macro.srdf.xacro (robot description, xacro)
@@ -39,5 +39,26 @@
       <joint name="${prefix}wrist_3_joint" value="-0.11" />
     </group_state>
+    <!-- |||||||||||||||||||||||||||||||||||||||||||||||||||||||||||||||||||||||||||||||||||||||||||||||||||||||||||||||||||||| -->
+    <group_state name="puntoA" group="${prefix}${name}_manipulator">
+      <joint name="${prefix}elbow_joint" value="0.889" />
+      <joint name="${prefix}shoulder_lift_joint" value="-0.497" />
+      <joint name="${prefix}shoulder_pan_joint" value="-2.089" />
+      <joint name="${prefix}wrist_1_joint" value="-0.364" />
+      <joint name="${prefix}wrist_2_joint" value="0.962" />
+      <joint name="${prefix}wrist_3_joint" value="1.558" />
+    </group_state>
+    <group_state name="puntoB" group="${prefix}${name}_manipulator">
+      <joint name="${prefix}elbow_joint" value="0.663" />
+      <joint name="${prefix}shoulder_lift_joint" value="-0.962" />
+      <joint name="${prefix}shoulder_pan_joint" value="-2.155" />
+      <joint name="${prefix}wrist_1_joint" value="-0.033" />
+      <joint name="${prefix}wrist_2_joint" value="1.624" />
+      <joint name="${prefix}wrist_3_joint" value="1.558" />
+    </group_state>
+    <!-- |||||||||||||||||||||||||||||||||||||||||||||||||||||||||||||||||||||||||||||||||||||||||||||||||||||||||||||||||||||| -->
     <!--END EFFECTOR - Purpose - Represent information about an end effector.-->
+    <end_effector name="${prefix}cama_effector" parent_link="${prefix}tool0" group="${prefix}${name}_manipulator">
+      <component name="cama_component" link="${prefix}cama_impresion" />
+    </end_effector>
     <!--VIRTUAL JOINT - Purpose - this element defines a virtual joint between a robot link and an external frame of reference (considered fixed with respect to the robot)-->
     <!--DISABLE COLLISIONS - By default it is assumed that any link of the robot could potentially come into collision with any other link in the robot. This tag disables collision checking between a specified pair of links. -->
@@ -53,4 +74,9 @@
     <disable_collisions link1="${prefix}wrist_1_link" link2="${prefix}wrist_3_link" reason="Never" />
     <disable_collisions link1="${prefix}wrist_2_link" link2="${prefix}wrist_3_link" reason="Adjacent" />
-  </xacro:macro>
+    <!-- |||||||||||||||||||||||||||||||||||||||||||||||||||||||||||||||||||||||||||||||||||||||||||||||||||||||||||||||||||||| -->
+    <disable_collisions link1="${prefix}cama_impresion" link2="${prefix}wrist_3_link" reason="Adjacent" />
+    <disable_collisions link1="${prefix}cama_impresion" link2="${prefix}wrist_2_link" reason="Never" />
+    <disable_collisions link1="${prefix}cama_impresion" link2="${prefix}wrist_1_link" reason="Never" />
+    <disable_collisions link1="${prefix}mesa" link2="${prefix}base_link" reason="Adjacent" />
+      </xacro:macro>
 </robot>

Commit message: FIX: cambios de los sistemas de referencias

File: src/Universal_Robots_ROS2_Description/urdf/ur_macro.xacro (robot description, xacro)
@@ -330,5 +330,5 @@
            link/frame) to introduce the necessary rotation over Z (of pi rad).
       -->
-      <origin xyz="0 0 0" rpy="0 0 ${pi}" />
+      <origin xyz="0 0 0" rpy="0 0 0" /> <!-- cambiado -->
     </joint>
     <joint name="${tf_prefix}shoulder_pan_joint" type="revolute">
@@ -438,5 +438,5 @@
     <link name="${tf_prefix}cama_impresion">
       <visual>
-        <origin xyz="0 0 0" rpy="0 ${-pi/2} 0 "/>
+        <origin xyz="-0.00098 -0.0103 0.083" rpy="0 ${-pi/2} 0 "/>
         <geometry>
           <mesh filename="file://$(find ur_description)/meshes/Escenas/Camas/cama_impresion.stl" scale="0.001 0.001 0.001"/>
@@ -447,5 +447,5 @@
       </visual>
       <collision>
-        <origin xyz="0 0 0" rpy="0 ${-pi/2} 0"/>
+        <origin xyz="-0.00098 -0.0103 0.083" rpy="0 ${-pi/2} 0"/>
         <geometry>
           <mesh filename="file://$(find ur_description)/meshes/Escenas/Camas/cama_impresion.stl" scale="0.001 0.001 0.001"/>
@@ -453,5 +453,5 @@
       </collision>
       <inertial>
-        <origin xyz="0 0 0" rpy="0 0 0"/>
+        <origin xyz="-0.00098 -0.0103 0.083" rpy="0 0 0"/>
         <mass value="${wrist_3_mass}"/>
         <inertia ixx="0.00079" ixy="0.0" ixz="0.0" iyy="0.00079" iyz="0.0" izz="0.00034"/>
@@ -497,5 +497,5 @@
       <parent link="${tf_prefix}tool0" />
       <child link="${tf_prefix}cama_impresion" />
-      <origin xyz="0 0 0.167" rpy="0 0 0" />
+      <origin xyz="0.00098 0.0103 0.084" rpy="0 0 0" />
       <axis xyz="0 0 1" />
     </joint>

File: src/Universal_Robots_ROS2_Driver/ur_moveit_config/srdf/ur_macro.srdf.xacro (robot description, xacro)
@@ -44,18 +44,26 @@
     <!-- |||||||||||||||||||||||||||||||||||||||||||||||||||||||||||||||||||||||||||||||||||||||||||||||||||||||||||||||||||||| -->
     <group_state name="puntoA" group="${prefix}${name}_manipulator">
-      <joint name="${prefix}elbow_joint" value="0.889" />
-      <joint name="${prefix}shoulder_lift_joint" value="-0.497" />
-      <joint name="${prefix}shoulder_pan_joint" value="-2.089" />
-      <joint name="${prefix}wrist_1_joint" value="-0.364" />
-      <joint name="${prefix}wrist_2_joint" value="0.962" />
+      <joint name="${prefix}elbow_joint" value="1.569" />
+      <joint name="${prefix}shoulder_lift_joint" value="-0.962" />
+      <joint name="${prefix}shoulder_pan_joint" value="1.624" />
+      <joint name="${prefix}wrist_1_joint" value="-0.63" />
+      <joint name="${prefix}wrist_2_joint" value="1.624" />
       <joint name="${prefix}wrist_3_joint" value="1.558" />
     </group_state>
     <group_state name="puntoB" group="${prefix}${name}_manipulator">
-      <joint name="${prefix}elbow_joint" value="0.663" />
-      <joint name="${prefix}shoulder_lift_joint" value="-0.962" />
-      <joint name="${prefix}shoulder_pan_joint" value="-2.155" />
-      <joint name="${prefix}wrist_1_joint" value="-0.033" />
+      <joint name="${prefix}elbow_joint" value="1.601" />
+      <joint name="${prefix}shoulder_lift_joint" value="-1.425" />
+      <joint name="${prefix}shoulder_pan_joint" value="1.624" />
+      <joint name="${prefix}wrist_1_joint" value="-0.431" />
       <joint name="${prefix}wrist_2_joint" value="1.624" />
       <joint name="${prefix}wrist_3_joint" value="1.558" />
+    </group_state>
+        <group_state name="INICIO_TRAYECTORIA" group="${prefix}${name}_manipulator">
+      <joint name="${prefix}elbow_joint" value="1.8266" />
+      <joint name="${prefix}shoulder_lift_joint" value="-1.2364" />
+      <joint name="${prefix}shoulder_pan_joint" value="1.6756" />
+      <joint name="${prefix}wrist_1_joint" value="-0.5656" />
+      <joint name="${prefix}wrist_2_joint" value="1.5628" />
+      <joint name="${prefix}wrist_3_joint" value="0.2846" />
     </group_state>
     <!-- |||||||||||||||||||||||||||||||||||||||||||||||||||||||||||||||||||||||||||||||||||||||||||||||||||||||||||||||||||||| -->

Commit message: FEAT: mejor aproximación del SR cama a vertice cubo

File: src/Universal_Robots_ROS2_Description/urdf/ur_macro.xacro (robot description, xacro)
@@ -438,5 +438,5 @@
     <link name="${tf_prefix}cama_impresion">
       <visual>
-        <origin xyz="-0.00098 -0.0103 0.083" rpy="0 ${-pi/2} 0 "/>
+        <origin xyz="-0.0103 -0.0103 0.083" rpy="0 ${-pi/2} 0 "/>
         <geometry>
           <mesh filename="file://$(find ur_description)/meshes/Escenas/Camas/cama_impresion.stl" scale="0.001 0.001 0.001"/>
@@ -447,5 +447,5 @@
       </visual>
       <collision>
-        <origin xyz="-0.00098 -0.0103 0.083" rpy="0 ${-pi/2} 0"/>
+        <origin xyz="-0.0103 -0.0103 0.083" rpy="0 ${-pi/2} 0"/>
         <geometry>
           <mesh filename="file://$(find ur_description)/meshes/Escenas/Camas/cama_impresion.stl" scale="0.001 0.001 0.001"/>
@@ -453,5 +453,5 @@
       </collision>
       <inertial>
-        <origin xyz="-0.00098 -0.0103 0.083" rpy="0 0 0"/>
+        <origin xyz="-0.0103 -0.0103 0.083" rpy="0 0 0"/>
         <mass value="${wrist_3_mass}"/>
         <inertia ixx="0.00079" ixy="0.0" ixz="0.0" iyy="0.00079" iyz="0.0" izz="0.00034"/>
@@ -497,5 +497,5 @@
       <parent link="${tf_prefix}tool0" />
       <child link="${tf_prefix}cama_impresion" />
-      <origin xyz="0.00098 0.0103 0.084" rpy="0 0 0" />
+      <origin xyz="0.0103 0.0103 0.084" rpy="0 0 0" />
       <axis xyz="0 0 1" />
     </joint>

Commit message: FEAT: añadido el brazo del extrusor en la simulación. SRDF + URDF

File: src/Universal_Robots_ROS2_Description/urdf/ur_macro.xacro (robot description, xacro)
@@ -436,4 +436,21 @@
       </collision>
     </link>
+    <link name="barra_extrusor">
+      <visual>
+        <origin xyz="0 0 0" rpy="0 0 ${pi/2}"/>
+        <geometry>
+          <mesh filename="file://$(find ur_description)/meshes/Escenas/barra_extrusor.stl" scale="0.0001 0.0001 0.0001"/>
+        </geometry>
+        <material name="GreyMetallic">
+          <color rgba="0.7 0.7 0.7 1.0"/>
+        </material>
+      </visual>
+      <collision>
+        <origin xyz="0 0 0" rpy="0 0 0"/>
+        <geometry>
+          <mesh filename="file://$(find ur_description)/meshes/Escenas/barra_extrusor.stl" scale="0.0001 0.0001 0.0001"/>
+        </geometry>
+      </collision>
+    </link>
     <link name="${tf_prefix}cama_impresion">
       <visual>
@@ -464,4 +481,9 @@
       <origin xyz="0.76884 -0.27794 -0.16726" rpy="-0.0054 -0.0053 0.0116"/>
       <axis xyz="0 0 1" />
+    </joint>
+    <joint name="barra_extrusor_joint" type="fixed">
+      <parent link="mesa" />
+      <child link="barra_extrusor" />
+      <origin xyz="-0.3 -0.68 0.36" rpy="0 ${-pi/2} 0" />
     </joint>
     <!-- |||||||||||||||||||||||||||||||||||||||||||||||||||||||||||||||||||||||||||||||||||||||||||||||||||||||||||||||||||||| -->

File: src/Universal_Robots_ROS2_Driver/ur_moveit_config/srdf/ur_macro.srdf.xacro (robot description, xacro)
@@ -81,21 +81,25 @@
     <disable_collisions link1="${prefix}base_link" link2="${prefix}base_link_inertia" reason="Adjacent" />
     <disable_collisions link1="${prefix}base_link_inertia" link2="${prefix}shoulder_link" reason="Adjacent" />
+    <disable_collisions link1="${prefix}shoulder_link" link2="${prefix}upper_arm_link" reason="Adjacent" />
+    <disable_collisions link1="${prefix}upper_arm_link" link2="${prefix}forearm_link" reason="Adjacent" />
+    <disable_collisions link1="${prefix}forearm_link" link2="${prefix}wrist_1_link" reason="Adjacent" />
+    <disable_collisions link1="${prefix}wrist_1_link" link2="${prefix}wrist_2_link" reason="Adjacent" />
+    <disable_collisions link1="${prefix}wrist_2_link" link2="${prefix}wrist_3_link" reason="Adjacent" />
+    <disable_collisions link1="${prefix}tool0" link2="${prefix}wrist_3_link" reason="Adjacent" />
+    <disable_collisions link1="${prefix}wrist_3_link" link2="cama_impresion" reason="Adjacent" />
+    <disable_collisions link1="cama_impresion" link2="${prefix}tool0" reason="Adjacent" />
+    <disable_collisions link1="mesa" link2="${prefix}base_link" reason="Adjacent" />
+    <disable_collisions link1="mesa" link2="${prefix}base_link_inertia" reason="Adjacent" />
+    <disable_collisions link1="mesa" link2="barra_extrusor" reason="Adjacent" />
+    <!-- |||||||||||||||||||||||||||||||||||||||||||||||||||||||||||||||||||||||||||||||||||||||||||||||||||||||||||||||||||||| -->
     <disable_collisions link1="${prefix}tool0" link2="${prefix}wrist_1_link" reason="Never" />
     <disable_collisions link1="${prefix}tool0" link2="${prefix}wrist_2_link" reason="Never" />
-    <disable_collisions link1="${prefix}tool0" link2="${prefix}wrist_3_link" reason="Adjacent" />
-    <disable_collisions link1="${prefix}forearm_link" link2="${prefix}upper_arm_link" reason="Adjacent" />
-    <disable_collisions link1="${prefix}forearm_link" link2="${prefix}wrist_1_link" reason="Adjacent" />
-    <disable_collisions link1="${prefix}shoulder_link" link2="${prefix}upper_arm_link" reason="Adjacent" />
-    <disable_collisions link1="${prefix}wrist_1_link" link2="${prefix}wrist_2_link" reason="Adjacent" />
     <disable_collisions link1="${prefix}wrist_1_link" link2="${prefix}wrist_3_link" reason="Never" />
-    <disable_collisions link1="${prefix}wrist_2_link" link2="${prefix}wrist_3_link" reason="Adjacent" />
-    <!-- |||||||||||||||||||||||||||||||||||||||||||||||||||||||||||||||||||||||||||||||||||||||||||||||||||||||||||||||||||||| -->
-    <disable_collisions link1="cama_impresion" link2="${prefix}tool0" reason="Adjacent" />
     <disable_collisions link1="cama_impresion" link2="${prefix}wrist_3_link" reason="Never" />
     <disable_collisions link1="cama_impresion" link2="${prefix}wrist_2_link" reason="Never" />
     <disable_collisions link1="cama_impresion" link2="${prefix}wrist_1_link" reason="Never" />
-    <disable_collisions link1="mesa" link2="${prefix}base_link" reason="Adjacent" />
-    <disable_collisions link1="mesa" link2="${prefix}base_link_inertia" reason="Never" />
     <disable_collisions link1="mesa" link2="${prefix}shoulder_link" reason="Default" />
+    <disable_collisions link1="barra_extrusor" link2="base_link_inertia" reason="Never" />
+    <disable_collisions link1="barra_extrusor" link2="shoulder_link" reason="Never" />
     </xacro:macro>
 </robot>
